File: solar/QLMPPT-1/supply.kicad_sch (KiCad schematic)
At the start: 10 parts, among them T3 "G1"

Commit message: Continuing QLMPPT-1
Other:
- note added: "TL431: Adjustable shunt voltage reference Vref = 2.495V Vka = 2.5V to 36V Ika = -100mA to +150mA Iref = 0.5 to 10mA Behaves like a regular diode between anode and cathode. Behaves like a turned-on bipolar transistor between cathode and anode, when the Ref input exceeds Vref. R29 = 10e3 R28 = 47e3 Vref = 2.495 divider = R29/(R28+R29) Vmin = Vref/divider = 14.2215"
Changed lines of the file:
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@@
     (stroke (width 0) (type default) (color 0 0 0 0))
+  )
+  (text "TL431: Adjustable shunt voltage reference\nVref = 2.495V\nVka = 2.5V to 36V\nIka = -100mA to +150mA\nIref = 0.5 to 10mA\n\nBehaves like a regular diode between anode and cathode.\nBehaves like a turned-on bipolar transistor between cathode and anode,\nwhen the Ref input exceeds Vref.\n\nR29 = 10e3\nR28 = 47e3\nVref = 2.495\ndivider = R29/(R28+R29)\nVmin = Vref/divider = 14.2215\n"
+    (at 85.725 113.03 0)
+    (effects (font (size 1.27 1.27)) (justify left bottom))
   )
   (text "U7: EG1192H DC/DC controller\nPin 1: V+\nPin 2: GND (input)\nPin 3: DCDC_ENABLE\nPin 4: n.c.\nPin 5: to R37\nPin 6: to choke L3\nPin 7: GND (output)\nPin 8: Feedback input\n\nR37: 100R between pins 5 and 6\nC27: bypass between pins 6 and 7\n\nC29: Elko, 100uF, 16V\nC30: same, but ceramic\n\nR46\n\nL3\nD8\n"
